File: vehicle-control-unit/lighting.sch (KiCad schematic (older format))
At the start: 17 parts, among them J7 Conn_01x03_Male, J8 Conn_01x03_Male, J9 Conn_02x06_Male_UnitPerRow, Q1 BC517, U3 ULN2803A

Commit message: Change value of rear turn signal resistors
Parts:
- R12, R13: value 150E -> 180E
Changed lines of the file:
@@
 Sheet 2 3
 Title "Earth Rover"
-Date "2020-06-07"
-Rev "7"
+Date "2020-08-05"
+Rev "9"
 Comp "Vijfendertig BVBA"
 Comment1 "Maarten De Munck"
@@
 P 4500 7850
 F 0 "R12" H 4570 7896 50  0000 L CNN
-F 1 "150E" H 4570 7805 50  0000 L CNN
+F 1 "180E" H 4570 7805 50  0000 L CNN
 F 2 "Resistor_THT:R_Axial_DIN0207_L6.3mm_D2.5mm_P10.16mm_Horizontal" V 4430 7850 50  0001 C CNN
 F 3 "~" H 4500 7850 50  0001 C CNN
@@
 P 5100 7850
 F 0 "R13" H 5170 7896 50  0000 L CNN
-F 1 "150E" H 5170 7805 50  0000 L CNN
+F 1 "180E" H 5170 7805 50  0000 L CNN
 F 2 "Resistor_THT:R_Axial_DIN0207_L6.3mm_D2.5mm_P10.16mm_Horizontal" V 5030 7850 50  0001 C CNN
 F 3 "~" H 5100 7850 50  0001 C CNN
